Commit message: add all files

File: IRB300_description/urdf/IRB300_description.urdf (robot description, URDF)
Before this commit: robot huichuan_arm, 7 links, 6 joints
Links:
- added link gripper, mass 1.6073; collision mesh filename=package://IRB300_description/meshes/gripper.STL; visual mesh filename=package://IRB300_description/meshes/gripper.STL
- added link world
- link link_0: geometry collision mesh filename=package://IRB300_description/meshes/link_0.STL; visual mesh filename=package://IRB300_description/meshes/link_0.STL
- link link_1: geometry collision mesh filename=package://IRB300_description/meshes/link_1.STL; visual mesh filename=package://IRB300_description/meshes/link_1.STL
- link link_2: mass 16.1900771502942 -> 17.7972686684801; geometry collision mesh filename=package://IRB300_description/meshes/link_2.STL; visual mesh filename=package://IRB300_description/meshes/link_2.STL
- link link_3: geometry collision mesh filename=package://IRB300_description/meshes/link_3.STL; visual mesh filename=package://IRB300_description/meshes/link_3.STL
- link link_4: geometry collision mesh filename=package://IRB300_description/meshes/link_4.STL; visual mesh filename=package://IRB300_description/meshes/link_4.STL
- link link_5: mass 0.51914 -> 0.519143539991011; geometry collision mesh filename=package://IRB300_description/meshes/link_5.STL; visual mesh filename=package://IRB300_description/meshes/link_5.STL
- link link_6: geometry collision mesh filename=package://IRB300_description/meshes/link_6.STL; visual mesh filename=package://IRB300_description/meshes/link_6.STL
Joints:
- added joint joint_7: type fixed, parent link_6, child gripper, origin xyz=0.0232 0 0 rpy=0.5605 -1.5708 -2.1316, axis 0 0 0
- added joint world_to_base_link=: type fixed, parent world, child link_0
- joint joint_1: limit lower=-1.484 upper=1.484 effort=0 velocity=3.84 -> lower=-1.484 upper=1.484 effort=-1 velocity=3.84
- joint joint_2: limit lower=-1.265 upper=0.681 effort=0 velocity=0 -> lower=-1.265 upper=0.681 effort=-1 velocity=3.665
- joint joint_3: limit lower=-0.619 upper=1.509 effort=0 velocity=0 -> lower=-0.619 upper=1.509 effort=-1 velocity=4.363
- joint joint_4: limit lower=-1.745 upper=1.745 effort=0 velocity=0 -> lower=-1.745 upper=1.745 effort=-1 velocity=5.236
- joint joint_5: limit lower=-1.047 upper=1.047 effort=0 velocity=0 -> lower=-1.047 upper=1.047 effort=-1 velocity=5.236
- joint joint_6: limit lower=-3.14 upper=3.14 effort=0 velocity=0 -> lower=-3.14 upper=3.14 effort=-1 velocity=7.854; type continuous -> revolute
